File: hardware/fluepboard/fluepdot.sch (KiCad schematic (older format))
At the start: 16 parts, among them J1 Screw_Terminal_01x02, J2 USB_C_Receptacle_USB2.0, J3 Conn_02x17_Odd_Even, J4 Screw_Terminal_01x05, SW1 SW_Push, U1 ESP32-WROOM-32

Commit message: Commit jlcpcb compatible version
Parts:
- removed J1: Screw_Terminal_01x02, TerminalBlock_Phoenix:TerminalBlock_Phoenix_PTSM-0,5-2-2,5-V-SMD_1x02-1MP_P2.50mm_Vertical, symbol Connector:Screw_Terminal_01x02
- removed J2: USB_C_Receptacle_USB2.0, HIROSE_CX70M-24P1:CX70M-24P1, symbol fluepdot:USB_C_Receptacle_USB2.0
- removed J4: Screw_Terminal_01x05, TerminalBlock_Phoenix:TerminalBlock_Phoenix_PTSM-0,5-5-2,5-V-SMD_1x05-1MP_P2.50mm_Vertical, symbol Connector:Screw_Terminal_01x05
- removed R1, R2: 5k1, Resistor_SMD:R_0805_2012Metric, symbol Device:R
- removed SW1: SW_Push, B3U-1000P:SW_B3U-1000P, symbol Switch:SW_Push
- added C11: 100nF, Capacitor_SMD:C_0603_1608Metric, symbol Device:C
- added IC8: SP3485EN, Package_SO:SOIC-8_3.9x4.9mm_P1.27mm, symbol Interface_UART:SP3485EN
- added J1: USB_B, Connector_USB:USB_B_OST_USB-B1HSxx_Horizontal, symbol Connector:USB_B
- added J2: Conn_01x10_Female, fluepdot:TerminalBlock_Phoenix_MPT-0,5-10-2.54_1x10_P2.54mm_Horizontal, symbol Connector:Conn_01x10_Female
- added LED1: LED1, Diode_SMD:D_0805_2012Metric, symbol Device:LED
- added LED2: LED2, Diode_SMD:D_0805_2012Metric, symbol Device:LED
- added R22, R23: 270, Resistor_SMD:R_0603_1608Metric, symbol Device:R
- added S1: TS-1187A-B-A-B, TS-1187A-B-A-B:TS1187ABAB, symbol TS-1187A-B-A-B:TS-1187A-B-A-B
- C1, C2: footprint Capacitor_SMD:C_0805_2012Metric -> Capacitor_SMD:C_0603_1608Metric; Description (none) -> MULTILAYER CERAMIC CAPACITORS MLCC - SMD/SMT 100NF 50V 0603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; Extended Part (none) -> 0; LCSC (none) -> C14663; Manufacturer (none) -> CC0603KRX7R9BB104
- ESP32: renamed from U1; LCSC (none) -> -
- R3: footprint Resistor_SMD:R_0805_2012Metric -> Resistor_SMD:R_0603_1608Metric; Description (none) -> CHIP RESISTOR - SURFACE MOUNT 10KOHMS ±1% 1/10W 0603 ROHS; Extended Part (none) -> 0; LCSC (none) -> C25804; Manufacturer (none) -> 0603WAF1002T5E
Connections:
- net +12V: no longer J3.29 (Pin_29)
- net +3V3: now also C11.1, IC8.8 (VCC)
- net EN: now also S1.A1 (COM_1)
- net GND: now also C11.2, IC8.5 (GND), J1.4 (GND), J1.5 (Shield), J2.2 (Pin_2), J2.3 (Pin_3), R22.2, R23.2, S1.C1 (NO_1)
- net USB2Serial/D+: now also J1.3 (D+)
- net USB2Serial/D-: now also J1.2 (D-)
- net USB2Serial/VBus: now also J1.1 (VBUS)
- net VFlipdot: now also J3.29 (Pin_29)
- net RS485_RTS: now reaches ESP32.10 (IO25)
- net RS485_RTS: now also IC8.2 (~RE~), IC8.3 (DE)
- net LED1: now reaches ESP32.26 (IO4)
- net LED1: now also LED1.1 (K)
- net LED2: now reaches ESP32.27 (IO16)
- net LED2: now also LED2.1 (K)
- net RS485_RXD: now reaches ESP32.36 (IO22)
- net RS485_RXD: now also IC8.1 (RO)
- net RS485_TXD: now reaches ESP32.37 (IO23)
- net RS485_TXD: now also IC8.4 (DI)
- new net: LED1.2 (A), R23.1
- new net: LED2.2 (A), R22.1
- new net RS485_A: IC8.6 (A), J2.5 (Pin_5)
- new net RS485_B: IC8.7 (B), J2.4 (Pin_4)
- new net SELECT0_OUT: J2.6 (Pin_6)
- new net SELECT1_OUT: J2.7 (Pin_7)
- new net SELECT2_OUT: J2.8 (Pin_8)
- new net SELECT3_OUT: J2.9 (Pin_9)
- new net SELECT4_OUT: J2.10 (Pin_10)
- new net V_in: J2.1 (Pin_1)
- no-connect marks 25 -> 20
Other:
- note added: "RS485"
